File: pcb/d3vk1t/d3vk1t.kicad_sch (KiCad schematic)
At the start: 4 parts

Commit message: project update  - update pcb layout.  - update schmatics sheets.  - added manufacturing files.  - added documentation files.
Other:
- sheet comm ports: added CAN1_RX, CAN1_TX, CAN_STB, RS485_DE, USART3_RX, USART3_TX; removed none
- sheet mcu ports: added ACC_CS, ACC_INT, BARO_CS, BUZZER, CAN1_RX, CAN1_TX, CAN_STB, I2C1_SCL, I2C1_SDA, RGB_B, RGB_G, RGB_R, RS485_DE, SDIO_CLK, SDIO_CMD, SDIO_D0, SDIO_D1, SDIO_D2, SDIO_D3, SDIO_DET, SPI1_CLK, SPI1_MISO, SPI1_MOSI, USART2_RX, USART2_TX, USART3_RX, USART3_TX, USB_N, USB_P; removed none
- sheet misc ports: added BUZZER, RGB_B, RGB_G, RGB_R; removed none
- sheet sdcard ports: added SDIO_CLK, SDIO_CMD, SDIO_D0, SDIO_D1, SDIO_D2, SDIO_D3, SDIO_DET; removed none
- sheet sensors ports: added ACC_CS, ACC_INT, BARO_CS, I2C1_SCL, I2C1_SDA, SPI1_CLK, SPI1_MISO, SPI1_MOSI; removed none
- sheet usb ports: added USB_N, USB_P; removed none
- sheet wifi_ble ports: added USART2_RX, USART2_TX; removed none
- title: (none) -> D3VK1T
- moved on the sheet: H1, H2, H3, H4
