File: pcb/d3vk1t/misc.kicad_sch (KiCad schematic)
At the start: 0 parts

Commit message: [update all schematics sheets]
Parts:
- added BZ1: Buzzer, Buzzer_Beeper:PUIAudio_SMT_0825_S_4_R, symbol Device:Buzzer
- added D1: LED_RGB, LED_SMD:LED_RGB_5050-6, symbol Device:LED_RGB
- added Q3: 2N7002, Package_TO_SOT_SMD:SOT-23-3, symbol Transistor_FET:2N7002
- added R3 (x4): 10K, Resistor_SMD:R_0402_1005Metric, symbol Device:R_Small
- added R3: 1K, Resistor_SMD:R_0402_1005Metric, symbol Device:R_Small
Connections:
- new net: D1.5 (GA), R3.1
- new net: BZ1.2 (+), Q3.3 (D), R3.1
- new net: D1.6 (RA), R3.1
- new net: D1.4 (BA), R3.1
- new net +5V: BZ1.1 (-), R3.2
- new net BUZZER: Q3.1 (G), R3.2
- new net GND: D1.1 (RK), D1.2 (GK), D1.3 (BK), Q3.2 (S), R3.1
- new net RGB_B: R3.2
- new net RGB_G: R3.2
- new net RGB_R: R3.2

Commit message: pcb: update layout
Parts:
- Q3: footprint Package_TO_SOT_SMD:SOT-23-3 -> bruno-libs:SOT-23B
Changed lines of the file:
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@@
       (effects (font (size 1.27 1.27)) (justify left))
     )
-    (property "Footprint" "Package_TO_SOT_SMD:SOT-23-3" (at 198.12 108.585 0)
+    (property "Footprint" "bruno-libs:SOT-23B" (at 198.12 108.585 0)
       (effects (font (size 1.27 1.27) italic) (justify left) hide)
     )

Commit message: project update  - update pcb layout.  - update schmatics sheets.  - added manufacturing files.  - added documentation files.
Parts:
- R3: value 10K -> 470R
- R3: value 10K -> 330R
- R3: value 10K -> 120R
Other:
- note added: "BUZZER"
- note added: "STATUS LED"
- title: (none) -> Miscellaneous
- moved on the sheet: BZ1, Q3, R3
