File: pcb/d3vk1t/usb.kicad_sch (KiCad schematic)
At the start: 0 parts

Commit message: [update all schematics sheets]
Parts:
- added C1: 1nF, Capacitor_SMD:C_1206_3216Metric, symbol Device:C_Small
- added C5 (x2): 100nF, Capacitor_SMD:C_0402_1005Metric, symbol Device:C_Small
- added C6 (x2): 1uF, Capacitor_SMD:C_0603_1608Metric, symbol Device:C_Small
- added IC: LM1117MP-3.3, Package_TO_SOT_SMD:SOT-223-3_TabPin2, symbol Regulator_Linear:LM1117MP-3.3
- added J6: 105450-0101, MOLEX_105450-0101, symbol db-usb:105450-0101
- added R3 (x2): 5.1K, Resistor_SMD:R_0402_1005Metric, symbol Device:R_Small
- added R3: 1M, Resistor_SMD:R_1206_3216Metric, symbol Device:R_Small
- added U4: USBLC6-2SC6, Package_TO_SOT_SMD:SOT-23-6, symbol Power_Protection:USBLC6-2SC6
Connections:
- new net: J6.A5 (CC1), R3.2
- new net: J6.A6 (D1+), J6.A7 (D1-)
- new net: J6.B5 (CC2), R3.2
- new net: J6.B6 (D2+), J6.B7 (D2-)
- new net: C1.1, J6.S1 (SHIELD), J6.S2 (SHIELD), J6.S3 (SHIELD), J6.S4 (SHIELD), R3.2
- new net +3.3V: C5.1, C6.1, IC.2 (VO)
- new net +5V: C5.1, C6.1, IC.3 (VI), J6.A4 (VBUS_A), J6.A9 (VBUS_A), J6.B4 (VBUS_B), J6.B9 (VBUS_B), U4.5 (VBUS)
- new net GND: C1.2, C5.2, C5.2, C6.2, C6.2, IC.1 (GND), J6.A1 (GND_A), J6.A12 (GND_A), J6.B1 (GND_B), J6.B12 (GND_B), R3.1, R3.1, R3.1, U4.2 (GND)
- no-connect marks 0 -> 10

Commit message: sch: update all sch sheets.
Parts:
- X1: renamed from J6; footprint MOLEX_105450-0101 -> db:MOLEX_105450-0101
- renumbered U4 to IC7, IC to IC8
Connections:
- net USB_CON_N: now reaches X1.A7 (D1-)
- net USB_CON_N: now also IC7.6 (I/O1), X1.B7 (D2-); no longer X1.A6 (D1+)
- net USB_CON_P: now reaches X1.B6 (D2+)
- net USB_CON_P: now also IC7.4 (I/O2), X1.A6 (D1+); no longer X1.B7 (D2-)
- net USB_N: now reaches IC7.1 (I/O1)
- net USB_P: now reaches IC7.3 (I/O2)
Changed lines of the file:
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@@
   (junction (at 91.44 58.42) (diameter 0) (color 0 0 0 0)
   )
-  (junction (at 86.36 68.58) (diameter 0) (color 0 0 0 0)
-  )
   (junction (at 30.48 99.06) (diameter 0) (color 0 0 0 0)
   )
@@
   )
   (junction (at 48.26 106.68) (diameter 0) (color 0 0 0 0)
-  )
-  (junction (at 86.36 73.66) (diameter 0) (color 0 0 0 0)
   )
   (junction (at 200.66 76.2) (diameter 0) (color 0 0 0 0)
@@
     (stroke (width 0) (type default))
   )
-  (wire (pts (xy 86.36 73.66) (xy 93.98 73.66))
-    (stroke (width 0) (type default))
-  )
-  (wire (pts (xy 81.28 165.1) (xy 88.9 165.1))
+  (wire (pts (xy 81.28 165.1) (xy 93.98 165.1))
     (stroke (width 0) (type default))
   )
@@
     (stroke (width 0) (type default))
   )
-  (wire (pts (xy 83.82 73.66) (xy 86.36 73.66))
-    (stroke (width 0) (type default))
-  )
   (wire (pts (xy 83.82 58.42) (xy 91.44 58.42))
     (stroke (width 0) (type default))
@@
     (stroke (width 0) (type default))
   )
-  (wire (pts (xy 86.36 71.12) (xy 86.36 73.66))
+  (wire (pts (xy 48.26 165.1) (xy 60.96 165.1))
     (stroke (width 0) (type default))
   )
@@
     (stroke (width 0) (type default))
   )
+  (wire (pts (xy 83.82 66.04) (xy 96.52 66.04))
+    (stroke (width 0) (type default))
+  )
+  (wire (pts (xy 83.82 71.12) (xy 96.52 71.12))
+    (stroke (width 0) (type default))
+  )
   (wire (pts (xy 83.82 101.6) (xy 99.06 101.6))
     (stroke (width 0) (type default))
@@
     (stroke (width 0) (type default))
   )
-  (wire (pts (xy 83.82 71.12) (xy 86.36 71.12))
-    (stroke (width 0) (type default))
-  )
   (wire (pts (xy 170.18 76.2) (xy 170.18 78.74))
     (stroke (width 0) (type default))
@@
     (stroke (width 0) (type default))
   )
+  (wire (pts (xy 83.82 73.66) (xy 96.52 73.66))
+    (stroke (width 0) (type default))
+  )
   (wire (pts (xy 50.8 104.14) (xy 48.26 104.14))
     (stroke (width 0) (type default))
@@
     (stroke (width 0) (type default))
   )
-  (wire (pts (xy 86.36 66.04) (xy 86.36 68.58))
-    (stroke (width 0) (type default))
-  )
   (wire (pts (xy 180.34 76.2) (xy 180.34 78.74))
     (stroke (width 0) (type default))
   )
-  (wire (pts (xy 81.28 170.18) (xy 88.9 170.18))
+  (wire (pts (xy 81.28 170.18) (xy 93.98 170.18))
     (stroke (width 0) (type default))
   )
@@
     (stroke (width 0) (type default))
   )
-  (wire (pts (xy 86.36 68.58) (xy 93.98 68.58))
-    (stroke (width 0) (type default))
-  )
   (wire (pts (xy 30.48 96.52) (xy 50.8 96.52))
     (stroke (width 0) (type default))
   )
-  (wire (pts (xy 53.34 165.1) (xy 60.96 165.1))
-    (stroke (width 0) (type default))
-  )
   (wire (pts (xy 30.48 114.3) (xy 38.1 114.3))
     (stroke (width 0) (type default))
@@
     (stroke (width 0) (type default))
   )
-  (wire (pts (xy 53.34 170.18) (xy 60.96 170.18))
-    (stroke (width 0) (type default))
-  )
-  (wire (pts (xy 83.82 68.58) (xy 86.36 68.58))
+  (wire (pts (xy 48.26 170.18) (xy 60.96 170.18))
     (stroke (width 0) (type default))
   )
@@
     (stroke (width 0) (type default))
   )
-  (wire (pts (xy 83.82 66.04) (xy 86.36 66.04))
-    (stroke (width 0) (type default))
-  )
   (wire (pts (xy 170.18 83.82) (xy 170.18 86.36))
     (stroke (width 0) (type default))
   )
+  (wire (pts (xy 83.82 68.58) (xy 96.52 68.58))
+    (stroke (width 0) (type default))
+  )
   (wire (pts (xy 91.44 104.14) (xy 83.82 104.14))
     (stroke (width 0) (type default))
@@
     (stroke (width 0) (type default))
   )
+  (label "USB_CON_P" (at 83.82 66.04 0) (fields_autoplaced)
+    (effects (font (size 1.27 1.27)) (justify left bottom))
+  )
+  (label "USB_CON_N" (at 48.26 165.1 0) (fields_autoplaced)
+    (effects (font (size 1.27 1.27)) (justify left bottom))
+  )
+  (label "USB_P" (at 83.82 170.18 0) (fields_autoplaced)
+    (effects (font (size 1.27 1.27)) (justify left bottom))
+  )
+  (label "USB_CON_N" (at 83.82 71.12 0) (fields_autoplaced)
+    (effects (font (size 1.27 1.27)) (justify left bottom))
+  )
+  (label "USB_N" (at 48.26 170.18 0) (fields_autoplaced)
+    (effects (font (size 1.27 1.27)) (justify left bottom))
+  )
+  (label "USB_CON_N" (at 83.82 68.58 0) (fields_autoplaced)
+    (effects (font (size 1.27 1.27)) (justify left bottom))
+  )
+  (label "USB_CON_P" (at 83.82 73.66 0) (fields_autoplaced)
+    (effects (font (size 1.27 1.27)) (justify left bottom))
+  )
+  (label "USB_CON_P" (at 83.82 165.1 0) (fields_autoplaced)
+    (effects (font (size 1.27 1.27)) (justify left bottom))
+  )
+  (global_label "USB_N" (shape bidirectional) (at 48.26 170.18 180) (fields_autoplaced)
+    (effects (font (size 1.27 1.27)) (justify right))
+    (property "Intersheetrefs" "${INTERSHEET_REFS}" (at 38.1348 170.18 0)
+      (effects (font (size 1.27 1.27)) (justify right) hide)
+    )
+  )
+  (global_label "USB_P" (shape bidirectional) (at 93.98 170.18 0) (fields_autoplaced)
+    (effects (font (size 1.27 1.27)) (justify left))
+    (property "Intersheetrefs" "${INTERSHEET_REFS}" (at 104.0447 170.18 0)
+      (effects (font (size 1.27 1.27)) (justify left) hide)
+    )
+  )
   (symbol (lib_name "105450-0101_1") (lib_id "db-usb:105450-0101") (at 15.24 114.3 0) (unit 1)
     (in_bom yes) (on_board yes) (dnp no) (fields_autoplaced)
-    (property "Reference" "J6" (at 67.31 46.99 0)
+    (property "Reference" "X1" (at 67.31 46.99 0)
       (effects (font (size 1.27 1.27)))
     )
@@
       (effects (font (size 1.27 1.27)))
     )
-    (property "Footprint" "MOLEX_105450-0101" (at 15.24 114.3 0)
+    (property "Footprint" "db:MOLEX_105450-0101" (at 15.24 114.3 0)
       (effects (font (size 1.27 1.27)) (justify bottom) hide)
     )
@@
       (project "d3vk1t"
         (path "/4ea523ae-7c45-478e-a9cc-6f4833d1a9d5/fd7cf4b0-4d20-445a-8ab6-186a5df83da1"
-          (reference "J6") (unit 1)
+          (reference "X1") (unit 1)
         )
       )
@@
   (symbol (lib_id "Regulator_Linear:LM1117MP-3.3") (at 190.5 76.2 0) (unit 1)
     (in_bom yes) (on_board yes) (dnp no) (fields_autoplaced)
-    (property "Reference" "IC" (at 190.5 69.85 0)
+    (property "Reference" "IC8" (at 190.5 69.85 0)
       (effects (font (size 1.27 1.27)))
     )
@@
       (project "d3vk1t"
         (path "/4ea523ae-7c45-478e-a9cc-6f4833d1a9d5/fd7cf4b0-4d20-445a-8ab6-186a5df83da1"
-          (reference "IC") (unit 1)
+          (reference "IC8") (unit 1)
         )
       )
@@
   (symbol (lib_id "Power_Protection:USBLC6-2SC6") (at 71.12 167.64 0) (unit 1)
     (in_bom yes) (on_board yes) (dnp no) (fields_autoplaced)
-    (property "Reference" "U4" (at 73.7617 156.21 0)
+    (property "Reference" "IC7" (at 73.7617 156.21 0)
       (effects (font (size 1.27 1.27)) (justify left))
     )
@@
       (project "d3vk1t"
         (path "/4ea523ae-7c45-478e-a9cc-6f4833d1a9d5/fd7cf4b0-4d20-445a-8ab6-186a5df83da1"
-          (reference "U4") (unit 1)
-        )
-      )
+          (reference "IC7") (unit 1)
+        )
+      )

Commit message: project update  - update pcb layout.  - update schmatics sheets.  - added manufacturing files.  - added documentation files.
Other:
- note added: "LDO 3.3V/0.8A"
- note added: "USB CONNECTOR"
- note added: "USB TVS"
- title: (none) -> USB
- moved on the sheet: C1, C5, C6, IC7, IC8, R3, X1
